File: ledSkateBoard.brd (EAGLE design)
At the start: 23 x 47.2 mm, 28 parts, among them J1 JST, U1 MPU-9150, U2 ATMEGA328P_TQFP, U4 MIC2505 3.3

Commit message: Final version before ordering.
Parts:
- removed C2, C3: 10uF, SparkFun-Capacitors:CAP-PTH-SMALL
- removed C4, C5, C6, C7: 4.7uF, SparkFun-Capacitors:CAP-PTH-SMALL
- removed C8: .1uF, SparkFun-Capacitors:CAP-PTH-SMALL
- removed R1, R2: 10K, SparkFun-Resistors:0603-RES
- removed R3: 330, SparkFun-Resistors:0603-RES
- removed R4: 2K, SparkFun-Resistors:0603-RES
- removed R5: 1K, SparkFun-Resistors:0603-RES
- removed R6: 4.3K, SparkFun-Resistors:0603-RES
- removed R7: 36K, SparkFun-Resistors:0603-RES
- removed TP1: TEST-POINT3, SparkFun-Passives:PAD.03X.03
- added C10, C11, C12, C9: 4.7uF, SparkFun-Capacitors:0805
- added C13: .1uF, SparkFun-Capacitors:0805
- added C14, C15, C17: 10uF, SparkFun-Capacitors:0805
- added R10: 36K, SparkFun-Resistors:0805
- added R11, R12: 10K, SparkFun-Resistors:0805
- added R13: 330, SparkFun-Resistors:0805
- added R14: 2K, SparkFun-Resistors:0805
- added R8: 1K, SparkFun-Resistors:0805
- added R9: 4.3K, SparkFun-Resistors:0805
- added TP3: TEST-POINT3, SparkFun-Passives:PAD.03X.03
- C1: device SparkFun-Capacitors:CAP-PTH-SMALL -> SparkFun-Capacitors:0805
- D2, D3: value RB751 -> Schottky .35Vf; device SparkFun-DiscreteSemi:SOD-523 -> microbuilder:SMADIODE
- moved D2 9.20 mm to (33.0, 4.32), flipped to the bottom, turned to 270 degrees
- moved D3 7.55 mm to (37.7, 4.19), flipped to the bottom, turned to 90 degrees
- moved C1 7.02 mm to (33.2, 18.0), turned to 0 degrees
Connections:
- net 5V: now also C9.1, R13.2; no longer C4.1, R3.2
- net GND: now also C1.1, C10.2, C11.2, C12.2, C13.1, C14.1, C15.1, C17.1, C9.2, R10.1, R14.1; no longer C1.2, C2.2, C3.2, C4.2, C5.2, C6.2, C7.2, C8.1, R4.1, R7.1
- net N$1: now also C11.1; no longer C6.1
- net N$11: now also R14.2; no longer R4.2
- net N$2: now also C12.1; no longer C7.1
- net N$3: now also C14.2; no longer C1.1
- net N$4: now also R10.2, R9.1, TP3.P$1; no longer R6.1, R7.2
- net N$7: now also R13.1; no longer R3.1
- net RESET: now also R8.1; no longer R5.1
- net SCL: now also R12.1; no longer R2.1
- net SDA: now also R11.1; no longer R1.1
- net VCC: now also C1.2, C13.2, C15.2, C17.2, R11.2, R12.2, R8.2; no longer C2.1, C3.1, C8.2, R1.2, R2.2, R5.2
- net V_BATT: now also C10.1, R9.2; no longer C5.1, R6.2
Routing:
- net 5V: track 14.1 -> 35.9 mm
- net GND: track 19.4 -> 31.4 mm, vias 1 -> 0
- net N$3: track 10.4 -> 20.8 mm, vias 0 -> 1
- net N$1: track 2.87 -> 7.99 mm, vias 0 -> 2
- net V_BATT: track 55.1 -> 59.4 mm
- net N$4: track 7.77 -> 5.13 mm
- net N$11: track 1.36 -> 3.33 mm
- net N$7: track 2.24 -> 4.13 mm
- net MPU_INT: track 15.0 -> 16.6 mm
- net SCL: track 10.4 -> 9.44 mm
- net RESET: track 24.8 -> 23.8 mm
- net N$2: track 2.41 -> 1.59 mm
- net VCC: track 68.3 -> 68.9 mm
Other:
- board size 23 x 47.2 mm -> 23 x 47.6 mm
- board text added: "10uF"
- board text added: "5V Power Jack"
- board text added: "DATA"
- board text added: "MCP73831"
- board text added: "MIC2505-3.3V"
- board text added: "MPU9150"

Commit message: Learned how to use Smash tool. Redid silkscreen
Parts:
- removed FRAME1: (no value), SparkFun-Aesthetics:CREATIVE_COMMONS
Routing:
- net N$8: track 9.57 -> 8.49 mm
Other:
- board text removed: "10uF"
- board text removed: "5V Power Jack"
- board text removed: "MCP73831"
- board text removed: "MIC2505-3.3V"

Commit message: First commit
Parts:
- removed D2, D3: Schottky .35Vf, microbuilder:SMADIODE
- removed JP2: POWER_JACKPTH, SparkFun-Connectors:POWER_JACK_PTH
Connections:
- removed net N$3: C14.2, D2.C, D3.C, U4.1, U4.3
- net 5V: no longer D2.A, JP2.PWR
- net GND: no longer JP2.GND, JP2.GNDBREAK
- net V_BATT: now also C14.2, U4.1, U4.3; no longer D3.A
Routing:
- net 5V: track 35.9 -> 9.51 mm
- net N$3: track 20.8 -> 0.00 mm, vias 1 -> 0
- net V_BATT: track 59.4 -> 57.5 mm
Changed lines of the file:
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@@
 <attribute name="VALUE" x="42.926" y="18.669" size="0.254" layer="27" rot="R180"/>
-</element>
-<element name="JP2" library="SparkFun-Connectors" package="POWER_JACK_PTH" value="POWER_JACKPTH" x="45.212" y="-2.794" smashed="yes">
-<attribute name="PROD_ID" value="CONN-08197" x="45.212" y="-2.794" size="1.778" layer="27" display="off"/>
-<attribute name="NAME" x="43.688" y="1.397" size="0.4064" layer="25"/>
-<attribute name="VALUE" x="43.688" y="0.635" size="0.4064" layer="27"/>
 </element>
 <element name="JP3" library="SparkFun-Connectors" package="1X03" value="LED CONNECTOR" x="50.8" y="45.212" smashed="yes" rot="R180">
@@
 </element>
 <element name="TP3" library="SparkFun-Passives" package="PAD.03X.03" value="TEST-POINT3" x="46.6725" y="33.3375"/>
-<element name="D2" library="microbuilder" package="SMADIODE" value="Schottky .35Vf" x="33.02" y="4.318" smashed="yes" rot="MR270">
-<attribute name="NAME" x="31.115" y="6.858" size="0.8128" layer="26" font="vector" ratio="18" rot="MR270"/>
-<attribute name="VALUE" x="35.306" y="6.858" size="0.4064" layer="28" font="vector" ratio="10" rot="MR270"/>
-</element>
-<element name="D3" library="microbuilder" package="SMADIODE" value="Schottky .35Vf" x="37.719" y="4.191" smashed="yes" rot="MR90">
-<attribute name="NAME" x="39.624" y="1.651" size="0.8128" layer="26" font="vector" ratio="18" rot="MR90"/>
-<attribute name="VALUE" x="35.433" y="1.651" size="0.4064" layer="28" font="vector" ratio="10" rot="MR90"/>
-</element>
 <element name="R8" library="SparkFun-Resistors" package="0805" value="1K" x="34.2138" y="23.9268" smashed="yes" rot="R270">
 <attribute name="NAME" x="33.0073" y="24.3078" size="0.4064" layer="25" rot="R270"/>
@@
 <contactref element="U1" pad="11"/>
 <contactref element="U1" pad="9"/>
-<contactref element="JP2" pad="GNDBREAK"/>
-<contactref element="JP2" pad="GND"/>
 <contactref element="JP3" pad="3"/>
 <polygon width="0.254" layer="1" isolate="0.3048">
@@
 <contactref element="JP3" pad="1"/>
 <wire x1="46.452" y1="15.306" x2="44.892" y2="15.306" width="0.254" layer="1"/>
-<contactref element="D3" pad="A"/>
 <wire x1="38.481" y1="9.2075" x2="37.592" y2="10.0965" width="0.254" layer="1"/>
 <wire x1="37.592" y1="10.0965" x2="36.068" y2="10.0965" width="0.254" layer="1"/>
@@
 <wire x1="38.481" y1="9.2075" x2="38.481" y2="13.716" width="0.254" layer="16"/>
 <wire x1="38.481" y1="13.716" x2="40.5765" y2="15.8115" width="0.254" layer="16"/>
-<wire x1="37.719" y1="6.5405" x2="37.719" y2="8.4455" width="0.254" layer="16"/>
 <wire x1="37.719" y1="8.4455" x2="38.481" y2="9.2075" width="0.254" layer="16"/>
 <contactref element="R9" pad="2"/>
@@
 <wire x1="41.656" y1="15.8115" x2="44.3865" y2="15.8115" width="0.254" layer="1"/>
 <wire x1="44.3865" y1="15.8115" x2="44.892" y2="15.306" width="0.254" layer="1"/>
+<contactref element="C14" pad="2"/>
+<contactref element="U4" pad="1"/>
+<contactref element="U4" pad="3"/>
+<wire x1="35.24" y1="13.4319" x2="33.34" y2="13.4319" width="0" layer="19" extent="1-1"/>
+<wire x1="38.481" y1="13.716" x2="35.24" y2="13.4319" width="0" layer="19" extent="1-16"/>
+<wire x1="33.5644" y1="9.525" x2="34.9885" y2="8.9535" width="0" layer="19" extent="1-1"/>
 </signal>
 <signal name="N$7">
@@
 </signal>
 <signal name="5V">
-<contactref element="JP2" pad="PWR"/>
 <contactref element="U$1" pad="4"/>
 <wire x1="49.252" y1="15.306" x2="47.982" y2="13.676" width="0.254" layer="1"/>
-<wire x1="47.982" y1="13.676" x2="45.212" y2="10.906" width="0.254" layer="1"/>
-<contactref element="D2" pad="A"/>
-<wire x1="33.02" y1="1.9685" x2="33.02" y2="1.27" width="0.254" layer="16"/>
-<wire x1="33.02" y1="1.27" x2="34.29" y2="0" width="0.254" layer="16"/>
-<wire x1="34.29" y1="0" x2="40.64" y2="0" width="0.254" layer="16"/>
-<wire x1="40.64" y1="0" x2="41.91" y2="1.27" width="0.254" layer="16"/>
-<wire x1="41.91" y1="1.27" x2="41.91" y2="7.604" width="0.254" layer="16"/>
-<wire x1="41.91" y1="7.604" x2="45.212" y2="10.906" width="0.254" layer="16"/>
 <contactref element="R13" pad="2"/>
 <contactref element="C9" pad="1"/>
 <wire x1="39.3175" y1="11.4935" x2="44.6245" y2="11.4935" width="0.254" layer="1"/>
-<wire x1="44.6245" y1="11.4935" x2="45.212" y2="10.906" width="0.254" layer="1"/>
 <wire x1="39.3175" y1="11.4935" x2="39.3175" y2="13.0175" width="0.254" layer="1"/>
 <wire x1="39.3175" y1="13.0175" x2="39.751" y2="13.451" width="0.254" layer="1"/>
-</signal>
-<signal name="N$3">
-<contactref element="U4" pad="1"/>
-<contactref element="U4" pad="3"/>
-<wire x1="35.24" y1="13.4319" x2="35.24" y2="11.618" width="0.254" layer="1"/>
-<wire x1="33.34" y1="13.4319" x2="33.34" y2="14.544" width="0.254" layer="1"/>
-<wire x1="33.34" y1="14.544" x2="33.528" y2="14.732" width="0.254" layer="1"/>
-<wire x1="33.528" y1="14.732" x2="35.052" y2="14.732" width="0.254" layer="1"/>
-<wire x1="35.052" y1="14.732" x2="35.306" y2="14.478" width="0.254" layer="1"/>
-<wire x1="35.306" y1="14.478" x2="35.306" y2="13.4979" width="0.254" layer="1"/>
-<wire x1="35.306" y1="13.4979" x2="35.24" y2="13.4319" width="0.254" layer="1"/>
-<contactref element="D2" pad="C"/>
-<contactref element="D3" pad="C"/>
-<wire x1="37.719" y1="1.8415" x2="37.5285" y2="1.8415" width="0.254" layer="16"/>
-<wire x1="37.5285" y1="1.8415" x2="33.02" y2="6.35" width="0.254" layer="16"/>
-<wire x1="33.02" y1="6.6675" x2="33.02" y2="6.35" width="0.254" layer="16"/>
-<wire x1="33.02" y1="6.6675" x2="33.02" y2="7.3025" width="0.254" layer="16"/>
-<wire x1="33.02" y1="7.3025" x2="34.6075" y2="8.89" width="0.254" layer="16"/>
-<wire x1="34.6075" y1="8.89" x2="34.6075" y2="10.9855" width="0.254" layer="16"/>
-<contactref element="C14" pad="2"/>
-<via x="34.6075" y="10.9855" extent="1-16" drill="0.508"/>
-<wire x1="34.6075" y1="10.9855" x2="35.24" y2="11.618" width="0.254" layer="1"/>
-<wire x1="33.5644" y1="9.525" x2="33.5644" y2="9.9424" width="0.254" layer="1"/>
-<wire x1="33.5644" y1="9.9424" x2="34.6075" y2="10.9855" width="0.254" layer="1"/>
+<wire x1="44.6245" y1="11.4935" x2="47.982" y2="13.676" width="0" layer="19" extent="1-1"/>
 </signal>
 <signal name="N$4">

Commit message: Final on revA
Parts:
- removed R10: 36K, SparkFun-Resistors:0805
- removed R9: 4.3K, SparkFun-Resistors:0805
- removed TP3: TEST-POINT3, SparkFun-Passives:PAD.03X.03
- added C2, C3: 22pF, SparkFun-Capacitors:1206
- added C4: 10uF, SparkFun-Capacitors:1206
- added D2: GREEN, SparkFun-LED:LED-1206
- added D3, D4: PMEG4005EJ, SparkFun-DiscreteSemi:SOD-323
- added FB1: (no value), microbuilder:0805
- added JP2: (no value), SparkFun-Connectors:1X06_LOCK
- added Q1: 16Mhz, adafruit:HC49/S
- added R1: 330, SparkFun-Passives:1206
- added R2: 37K, SparkFun-Passives:1206
- added R3: 430K, SparkFun-Passives:1206
- added U3: (no value), adafruit:FGPMMOPA6H
- C1: value 10uF -> 10nF; device SparkFun-Capacitors:0805 -> SparkFun-Capacitors:1206
- C10, C13, C14, C15, C17, C9: device SparkFun-Capacitors:0805 -> SparkFun-Capacitors:1206
- C11: value 4.7uF -> .1uF; device SparkFun-Capacitors:0805 -> SparkFun-Capacitors:1206
- C12: value 4.7uF -> 2.2nF 50V; device SparkFun-Capacitors:0805 -> SparkFun-Capacitors:1206
- D1: device SparkFun-LED:LED-0603 -> SparkFun-LED:LED-1206
- JP3: value LED CONNECTOR -> M02LOCK; device SparkFun-Connectors:1X03 -> SparkFun-Connectors:1X02_LOCK
- R11, R12: value 10K -> 4.7K; device SparkFun-Resistors:0805 -> SparkFun-Passives:1206
- R13, R14, R8: device SparkFun-Resistors:0805 -> SparkFun-Passives:1206
- moved JP1 35.3 mm to (66.7, 41.0), turned to 180 degrees
- moved C11 29.8 mm to (56.6, 19.6), turned to 0 degrees
- moved D1 27.0 mm to (61.3, 2.54), flipped to the bottom, turned to 90 degrees
- moved JP3 26.0 mm to (46.1, 19.7), turned to 270 degrees
- moved R8 25.7 mm to (59.9, 22.5)
- moved C10 25.3 mm to (62.3, 7.98), flipped to the bottom, turned to 90 degrees
- moved C12 25.3 mm to (59.2, 23.0), flipped to the bottom, turned to 270 degrees
- moved C15 23.0 mm to (55.0, 17.2), flipped to the bottom, turned to 0 degrees
- moved C14 22.9 mm to (54.9, 14.9), flipped to the bottom, turned to 180 degrees
- moved U1 22.4 mm to (55.1, 24.1), turned to 0 degrees
- moved R13 22.1 mm to (58.6, 2.48), flipped to the bottom, turned to 90 degrees
- moved C13 21.3 mm to (48.6, 22.9)
- moved C9 20.4 mm to (60.1, 12.2), flipped to the bottom, turned to 180 degrees
- moved C1 18.8 mm to (50.9, 24.2), turned to 270 degrees
- moved C17 17.3 mm to (48.3, 34.2)
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Connections:
- removed net DATA: JP3.2, U2.12
- removed net MPU_INT: U1.12, U2.32
- new net AN0: JP2.2, U2.10
- new net AN1: JP2.3, U2.11
- new net GPS_RX: JP3.2, U2.31, U3.P$10
- new net GPS_TX: JP3.1, U2.30, U3.P$9
- new net N$10: C14.2, D3.C, D4.C, U4.1, U4.3
- new net N$3: C2.1, Q1.2, U2.7
- new net N$5: C3.1, Q1.1, U2.8
- new net N$6: D2.A, U3.P$5
- new net N$9: D2.C, R1.1
- new net PB0: JP2.4
- new net PB1: JP2.5, U2.13
- new net PB2: JP2.6, U2.14
- new net PD5: JP2.1, U2.9
- new net PWR_MNTR: R2.1, R3.2, U2.23
- net 5V: now also D3.A, JP1.2
- net GND: now also C2.2, C3.2, C4.2, R1.2, R3.1, U3.P$19, U3.P$3, U3.P$8; no longer JP3.3, R10.1
- net N$4: now also C4.1, FB1.1, U3.P$1; no longer R10.2, R9.1, TP3.P$1, U2.23
- net VCC: now also FB1.2; no longer JP1.2
- net V_BATT: now also D4.A, R2.2; no longer C14.2, JP3.1, R9.2, U4.1, U4.3
Routing:
- net 5V: track 9.51 -> 48.1 mm, vias 0 -> 2
- net DATA: track 24.7 -> 0.00 mm, vias 1 -> 0
- net V_BATT: track 57.5 -> 32.8 mm, vias 3 -> 0
- net GPS_RX: track 0.00 -> 20.5 mm, vias 0 -> 2
- net GPS_TX: track 0.00 -> 20.0 mm, vias 0 -> 2
- net MPU_INT: track 16.6 -> 0.00 mm
- net N$3: track 0.00 -> 14.6 mm
- net PWR_MNTR: track 0.00 -> 13.8 mm, vias 0 -> 1
- net N$6: track 0.00 -> 12.5 mm
- net MISO: track 9.57 -> 20.5 mm, vias 0 -> 1
- net VCC: track 68.9 -> 58.3 mm, vias 4 -> 2
- net N$10: track 0.00 -> 10.6 mm
- net N$5: track 0.00 -> 10.4 mm
- net PB2: track 0.00 -> 9.59 mm
- net MOSI: track 5.05 -> 13.5 mm, vias 0 -> 1
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Other:
- board size 23 x 47.6 mm -> 24.9 x 43.3 mm
- board text removed: "DATA"
- board text removed: "MPU9150"

Commit message: Final
Parts:
- moved C4 4.22 mm to (65.9, 16.3), turned to 270 degrees
- moved J1 3.84 mm to (48.6, 3.17)
- moved D1 2.79 mm to (63.8, 1.14), turned to 180 degrees
- moved C13 2.74 mm to (46.1, 23.9)
- moved R14 2.44 mm to (67.3, 8.45)
- moved C10 2.22 mm to (64.5, 8.48)
- moved C15 1.83 mm to (56.0, 18.7)
- moved R13 1.83 mm to (57.6, 0.95), turned to 0 degrees
- moved C14 1.63 mm to (55.9, 16.1)
- moved FB1 1.40 mm to (63.5, 20.2)
- moved D3 1.09 mm to (56.0, 12.8)
- moved D4 1.09 mm to (53.6, 12.8)
- moved U$1 1.02 mm to (60.6, 8.13)
- moved C11 0.64 mm to (56.6, 18.9)
- moved R12 0.36 mm to (47.1, 30.3)
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Routing:
- net V_BATT: track 32.8 -> 39.7 mm
- net N$8: track 2.83 -> 8.25 mm
- net VCC: track 58.3 -> 62.2 mm
- net 5V: track 48.1 -> 50.5 mm
- net N$11: track 5.80 -> 7.10 mm
- net PWR_MNTR: track 13.8 -> 14.9 mm
- net N$10: track 10.6 -> 11.3 mm
- net RESET: track 25.2 -> 24.6 mm
- net SCL: track 9.70 -> 10.3 mm
- net N$1: track 2.65 -> 3.23 mm
