File: ledSkateBoard.sch (EAGLE design)
At the start: 28 parts, among them J1 JST, U4 MIC2505 3.3

Commit message: Initial design
Parts:
- removed SDCARD: MICROSD, adafruit:MICROSD
- added JP2: (no value), microbuilder:JUMPER2
- added U2: (no value), Matts-Parts:W25Q128FV
Connections:
- removed net SD_CS: SDCARD.CS, U1.PIO0_2/SSEL0/CT16B0_CAP0
- removed net SD_DETECT: SDCARD.CARD_DETECT
- removed net SD_DI: SDCARD.DATA_IN, U1.PIO0_9/MOSI0/CT16B0_MAT1
- removed net SD_DO: SDCARD.DATA_OUT, U1.PIO0_8/MISO0/CT16B0_MAT0
- removed net SD_SCK: SDCARD.SCLK, U1.PIO0_6/SCK0
- new net N$10: JP2.2, MTK339.VCC
- new net WS_CS: U1.PIO0_2/SSEL0/CT16B0_CAP0, U2.CS
- new net WS_DI: U1.PIO0_9/MOSI0/CT16B0_MAT1, U2.DI
- new net WS_DO: U1.PIO0_8/MISO0/CT16B0_MAT0, U2.DO
- new net WS_RESET: U2.RESET
- new net WS_SCK: U1.PIO0_6/SCK0, U2.CLK
- net GND: now also U2.GND; no longer SDCARD.GND, SDCARD.GND1, SDCARD.VSS
- net N$4: now also JP2.1; no longer MTK339.VCC
- net VCC: now also U2.VCC; no longer SDCARD.VDD
Other:
- moved on the sheet: C3, FB1

Commit message: Closer..
Parts:
- removed J1: JST, SparkFun-Connectors:JST_2MM_MALE
- added BAT_CON: 53261-02, con-molex:53261-02
- C15, C4, C8: value 10uF -> .1uF
- FB1: value (none) -> GetValue
- renumbered JP1 to PROG_HEADER, U1 to W25Q128FV
Connections:
- removed net N$5: R8.2, W25Q128FV.PIO0_5/SDA
- removed net N$7: R4.1
- removed net N$8: R7.2, W25Q128FV.PIO0_4/SCL
- removed net WS_RESET: U2.RESET
- net GND: now also BAT_CON-1.S, R4.1; no longer J1.-
- net SCL: now also R8.2, W25Q128FV.PIO0_4/SCL
- net SDA: now also R7.2, W25Q128FV.PIO0_5/SDA
- net VCC: now also U2.RESET, U2.WP
- net V_BATT: now also BAT_CON-2.S; no longer J1.+
Other:
- moved on the sheet: R7, R8
