File: ProSense.brd (EAGLE design)
At the start: 25.5 x 36.7 mm, 24 parts, among them U4 MIC2505 3.3

Commit message: fixup
Routing:
- net VCC: track 92.7 -> 93.3 mm
Changed lines of the file:
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@@
 <layers>
 <layer number="1" name="Top" color="4" fill="1" visible="yes" active="yes"/>
-<layer number="16" name="Bottom" color="1" fill="1" visible="yes" active="yes"/>
+<layer number="16" name="Bottom" color="1" fill="1" visible="no" active="yes"/>
 <layer number="17" name="Pads" color="2" fill="1" visible="yes" active="yes"/>
 <layer number="18" name="Vias" color="2" fill="1" visible="yes" active="yes"/>
@@
 <layer number="20" name="Dimension" color="15" fill="1" visible="yes" active="yes"/>
 <layer number="21" name="tPlace" color="16" fill="1" visible="yes" active="yes"/>
-<layer number="22" name="bPlace" color="14" fill="1" visible="yes" active="yes"/>
+<layer number="22" name="bPlace" color="14" fill="1" visible="no" active="yes"/>
 <layer number="23" name="tOrigins" color="15" fill="1" visible="yes" active="yes"/>
-<layer number="24" name="bOrigins" color="15" fill="1" visible="yes" active="yes"/>
+<layer number="24" name="bOrigins" color="15" fill="1" visible="no" active="yes"/>
 <layer number="25" name="tNames" color="7" fill="1" visible="yes" active="yes"/>
-<layer number="26" name="bNames" color="7" fill="1" visible="yes" active="yes"/>
+<layer number="26" name="bNames" color="7" fill="1" visible="no" active="yes"/>
 <layer number="27" name="tValues" color="7" fill="1" visible="no" active="yes"/>
 <layer number="28" name="bValues" color="7" fill="1" visible="no" active="yes"/>
@@
 <layer number="110" name="fp0" color="7" fill="1" visible="no" active="yes"/>
 <layer number="111" name="LPC17xx" color="7" fill="1" visible="no" active="yes"/>
-<layer number="112" name="tSilk" color="7" fill="1" visible="yes" active="yes"/>
+<layer number="112" name="tSilk" color="7" fill="1" visible="no" active="yes"/>
 <layer number="113" name="IDFDebug" color="7" fill="1" visible="no" active="yes"/>
 <layer number="114" name="FRNTMAAT1" color="7" fill="1" visible="no" active="yes"/>
@@
 <wire x1="49.18945" y1="53.23905" x2="50.408" y2="54.4576" width="0.2032" layer="16"/>
 <wire x1="49.30775" y1="40.14935" x2="52.148" y2="40.14935" width="0.254" layer="16"/>
-<wire x1="52.148" y1="40.14935" x2="52.16875" y2="40.1701" width="0.254" layer="16"/>
-<wire x1="52.16875" y1="40.1701" x2="52.20685" y2="40.132" width="0.254" layer="16"/>
+<wire x1="52.148" y1="40.14935" x2="51.91475" y2="40.1701" width="0.254" layer="16"/>
+<wire x1="51.91475" y1="40.1701" x2="52.20685" y2="40.132" width="0.254" layer="16"/>
 <wire x1="52.20685" y1="40.132" x2="54.45125" y2="40.16375" width="0.254" layer="16"/>
 <wire x1="54.45125" y1="40.16375" x2="55.68315" y2="38.93185" width="0.254" layer="16"/>
-<wire x1="55.68315" y1="38.93185" x2="57.36875" y2="38.9001" width="0.254" layer="16"/>
-<wire x1="57.36875" y1="38.9001" x2="57.36875" y2="37.6301" width="0.254" layer="16"/>
-<wire x1="57.36875" y1="37.6301" x2="57.62795" y2="37.3709" width="0.254" layer="16"/>
+<wire x1="55.68315" y1="38.93185" x2="57.62275" y2="38.9001" width="0.254" layer="16"/>
+<wire x1="57.62275" y1="38.9001" x2="57.62275" y2="37.6301" width="0.254" layer="16"/>
+<wire x1="57.62275" y1="37.6301" x2="57.62795" y2="37.3709" width="0.254" layer="16"/>
 <wire x1="57.62795" y1="37.3709" x2="57.62795" y2="35.04565" width="0.254" layer="16"/>
 <wire x1="39.09695" y1="38.3899" x2="39.08595" y2="38.30565" width="0.254" layer="1"/>
@@
 <contactref element="W25Q128FV" pad="1"/>
 <contactref element="MCU" pad="19"/>
-<wire x1="52.16875" y1="37.6301" x2="52.20685" y2="37.592" width="0.254" layer="16"/>
+<wire x1="51.91475" y1="37.6301" x2="52.20685" y2="37.592" width="0.254" layer="16"/>
 <via x="54.32425" y="37.49675" extent="1-16" drill="0.508"/>
 <wire x1="54.0258" y1="35.3185" x2="54.0258" y2="36.40455" width="0.254" layer="1"/>
@@
 <contactref element="W25Q128FV" pad="2"/>
 <contactref element="MCU" pad="1"/>
-<wire x1="52.16875" y1="38.9001" x2="52.20685" y2="38.862" width="0.254" layer="16"/>
+<wire x1="51.91475" y1="38.9001" x2="52.20685" y2="38.862" width="0.254" layer="16"/>
 <wire x1="52.20685" y1="38.862" x2="54.102" y2="38.862" width="0.254" layer="16"/>
 <via x="54.102" y="38.862" extent="1-16" drill="0.508"/>
@@
 <wire x1="49.276" y1="42.291" x2="53.6575" y2="42.291" width="0.254" layer="16"/>
 <wire x1="53.6575" y1="42.291" x2="55.7784" y2="40.1701" width="0.254" layer="16"/>
-<wire x1="55.7784" y1="40.1701" x2="57.36875" y2="40.1701" width="0.254" layer="16"/>
+<wire x1="55.7784" y1="40.1701" x2="57.62275" y2="40.1701" width="0.254" layer="16"/>
 </signal>
 <signal name="WS_DI">
@@
 <via x="54.102" y="43.18" extent="1-16" drill="0.508"/>
 <wire x1="54.102" y1="43.18" x2="55.8419" y2="41.4401" width="0.254" layer="16"/>
-<wire x1="55.8419" y1="41.4401" x2="57.36875" y2="41.4401" width="0.254" layer="16"/>
+<wire x1="55.8419" y1="41.4401" x2="57.62275" y2="41.4401" width="0.254" layer="16"/>
 </signal>
 <signal name="N$10">

Commit message: fixup
Parts:
- removed PROGHEADER: (no value), SparkFun-Connectors:1X06_LOCK
- added U$1: DF13-6P-1.25H, con-hirose-df13:DF13A-6P-1.25H
Connections:
- net GND: now also U$1.P$3; no longer PROGHEADER.4
- net ISP: now also U$1.P$1; no longer PROGHEADER.6
- net LPC_RX: now also U$1.P$6; no longer PROGHEADER.1
- net LPC_TX: now also U$1.P$5; no longer PROGHEADER.2
- net RESET: now also U$1.P$2; no longer PROGHEADER.5
- net VCC: now also U$1.P$4; no longer PROGHEADER.3
Routing:
- net VCC: track 93.3 -> 88.4 mm
- net LPC_RX: track 25.7 -> 20.8 mm
- net LPC_TX: track 26.5 -> 21.9 mm
- net RESET: track 4.39 -> 0.00 mm
Changed lines of the file:
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@@
 <attribute name="VALUE" x="46.186" y="59.103" size="1.27" layer="28" rot="MR0"/>
-</element>
-<element name="PROGHEADER" library="SparkFun-Connectors" package="1X06_LOCK" value="" x="42.0751" y="31.242" smashed="yes">
-<attribute name="NAME" x="40.259" y="29.7561" size="0.4064" layer="25" font="vector" rot="R90"/>
-<attribute name="VALUE" x="40.8051" y="27.94" size="1.27" layer="27" font="vector"/>
 </element>
 <element name="MCU" library="NXP_60_26022015" package="SOT163-1" value="LPC1112FD20/102" x="49.5808" y="40.0685" smashed="yes" rot="R180">
@@
 <attribute name="NAME" x="49.8579" y="38.2176" size="0.4064" layer="25" font="vector" rot="R180"/>
 </element>
+<element name="U$1" library="con-hirose-df13" package="DF13A-6P-1.25H" value="DF13-6P-1.25H" x="48.133" y="26.035" rot="R180"/>
 </elements>
 <signals>
@@
 <contactref element="MCU" pad="15"/>
 <contactref element="C8" pad="1"/>
-<contactref element="PROGHEADER" pad="3"/>
-<wire x1="47.1551" y1="31.242" x2="47.1551" y2="31.9151" width="0.4064" layer="1"/>
-<wire x1="47.1551" y1="31.9151" x2="48.895" y2="33.655" width="0.4064" layer="1"/>
-<wire x1="48.895" y1="33.655" x2="48.895" y2="35.2677" width="0.4064" layer="1"/>
-<wire x1="48.895" y1="35.2677" x2="48.9458" y2="35.3185" width="0.4064" layer="1"/>
 <wire x1="53.07165" y1="60.52435" x2="55.73475" y2="60.52435" width="0.4064" layer="16"/>
 <wire x1="55.73475" y1="60.52435" x2="55.8292" y2="60.6188" width="0.4064" layer="16"/>
@@
 <wire x1="39.09695" y1="38.3899" x2="39.08595" y2="38.30565" width="0.254" layer="1"/>
 <via x="39.08425" y="34.00425" extent="1-16" drill="0.508"/>
-<wire x1="47.1551" y1="31.3309" x2="47.1551" y2="31.242" width="0.254" layer="16"/>
 <wire x1="37.40785" y1="45.92785" x2="37.8333" y2="45.9469" width="0.254" layer="1"/>
 <wire x1="37.8333" y1="45.9469" x2="40.64635" y2="45.9469" width="0.254" layer="1"/>
@@
 <wire x1="39.90975" y1="48.79975" x2="39.90975" y2="52.35325" width="0.4064" layer="1"/>
 <wire x1="39.90975" y1="52.35325" x2="39.05" y2="53.213" width="0.4064" layer="1"/>
+<contactref element="U$1" pad="P$4"/>
+<wire x1="40.59695" y1="38.3899" x2="42.83245" y2="40.14935" width="0" layer="19" extent="1-16"/>
+<wire x1="47.508" y1="26.935" x2="47.1551" y2="31.3309" width="0" layer="19" extent="1-16"/>
 </signal>
 <signal name="GND">
@@
 <contactref element="MCU" pad="16"/>
 <contactref element="C8" pad="2"/>
-<contactref element="PROGHEADER" pad="4"/>
 <wire x1="51.18945" y1="51.8427" x2="51.18945" y2="51.0402" width="0.254" layer="16"/>
 <wire x1="51.18945" y1="51.0402" x2="51.30195" y2="50.9277" width="0.254" layer="16"/>
@@
 <wire x1="49.75225" y1="49.9745" x2="51.25515" y2="49.9745" width="0.2032" layer="16"/>
 <wire x1="51.25515" y1="49.9745" x2="51.30195" y2="49.9277" width="0.2032" layer="16"/>
+<contactref element="U$1" pad="P$3"/>
+<wire x1="55.8292" y1="62.4188" x2="58.1423" y2="61.1378" width="0" layer="19" extent="1-16"/>
+<wire x1="52.391" y1="49.523" x2="51.30195" y2="49.9277" width="0" layer="19" extent="1-16"/>
+<wire x1="44.891" y1="49.523" x2="46.57695" y2="49.4277" width="0" layer="19" extent="1-16"/>
+<wire x1="53.891" y1="64.523" x2="55.8292" y2="62.4188" width="0" layer="19" extent="1-16"/>
+<wire x1="50.2158" y1="35.3185" x2="49.30775" y2="38.34935" width="0" layer="19" extent="1-16"/>
+<wire x1="43.391" y1="64.523" x2="42.936" y2="59.603" width="0" layer="19" extent="1-16"/>
+<wire x1="38.7079" y1="50.36185" x2="43.73415" y2="53.42255" width="0" layer="19" extent="1-16"/>
+<wire x1="58.028" y1="52.7812" x2="52.208" y2="54.4576" width="0" layer="19" extent="1-16"/>
+<wire x1="48.758" y1="26.935" x2="50.2158" y2="35.3185" width="0" layer="19" extent="1-1"/>
+<wire x1="40.88595" y1="35.66795" x2="49.30775" y2="38.34935" width="0" layer="19" extent="1-16"/>
+<wire x1="37.59695" y1="39.8399" x2="40.88595" y2="35.66795" width="0" layer="19" extent="1-1"/>
 </signal>
 <signal name="N$6">
@@
 <contactref element="MTK339" pad="P$9"/>
 <contactref element="MCU" pad="11"/>
-<contactref element="PROGHEADER" pad="1"/>
-<wire x1="43.8658" y1="35.3185" x2="43.8658" y2="34.3408" width="0.3048" layer="1"/>
-<wire x1="43.8658" y1="34.3408" x2="42.06875" y2="32.54375" width="0.3048" layer="1"/>
-<wire x1="42.06875" y1="32.54375" x2="42.06875" y2="31.24835" width="0.3048" layer="1"/>
-<wire x1="42.06875" y1="31.24835" x2="42.0751" y2="31.242" width="0.3048" layer="1"/>
 <via x="43.815" y="41.529" extent="1-16" drill="0.508"/>
 <wire x1="43.815" y1="41.529" x2="49.05375" y2="46.38675" width="0.254" layer="16"/>
@@
 <wire x1="43.8658" y1="35.3185" x2="43.8658" y2="41.4782" width="0.254" layer="1"/>
 <wire x1="43.8658" y1="41.4782" x2="43.815" y2="41.529" width="0.254" layer="1"/>
+<contactref element="U$1" pad="P$6"/>
+<wire x1="45.008" y1="26.935" x2="43.8658" y2="35.3185" width="0" layer="19" extent="1-1"/>
 </signal>
 <signal name="LPC_TX">
 <contactref element="MTK339" pad="P$10"/>
 <contactref element="MCU" pad="12"/>
-<contactref element="PROGHEADER" pad="2"/>
-<wire x1="44.6151" y1="30.988" x2="44.6151" y2="32.2326" width="0.3048" layer="1"/>
-<wire x1="44.6151" y1="32.2326" x2="45.085" y2="32.7025" width="0.3048" layer="1"/>
-<wire x1="45.085" y1="32.7025" x2="45.085" y2="35.2677" width="0.3048" layer="1"/>
-<wire x1="45.085" y1="35.2677" x2="45.1358" y2="35.3185" width="0.3048" layer="1"/>
 <wire x1="45.1358" y1="35.3185" x2="45.212" y2="35.3947" width="0.254" layer="1"/>
 <wire x1="45.212" y1="35.3947" x2="45.212" y2="41.275" width="0.254" layer="1"/>
@@
 <wire x1="55.372" y1="47.244" x2="55.391" y2="46.882" width="0.254" layer="1"/>
 <wire x1="55.391" y1="46.882" x2="55.391" y2="49.523" width="0.254" layer="1"/>
+<contactref element="U$1" pad="P$5"/>
+<wire x1="46.258" y1="26.935" x2="45.1358" y2="35.3185" width="0" layer="19" extent="1-1"/>
 </signal>
 <signal name="N$3">
@@
 <signal name="ISP">
 <contactref element="MCU" pad="18"/>
-<contactref element="PROGHEADER" pad="6"/>
 <wire x1="52.7558" y1="35.3185" x2="52.7558" y2="33.9217" width="0.3048" layer="1"/>
 <wire x1="52.7558" y1="33.9217" x2="54.76875" y2="31.90875" width="0.3048" layer="1"/>
 <wire x1="54.76875" y1="31.90875" x2="54.76875" y2="30.99435" width="0.3048" layer="1"/>
-<wire x1="54.76875" y1="30.99435" x2="54.7751" y2="30.988" width="0.3048" layer="1"/>
+<contactref element="U$1" pad="P$1"/>
+<wire x1="51.258" y1="26.935" x2="52.7558" y2="33.9217" width="0" layer="19" extent="1-1"/>
 </signal>
 <signal name="RESET">
 <contactref element="MCU" pad="17"/>
-<contactref element="PROGHEADER" pad="5"/>
-<wire x1="52.2351" y1="31.242" x2="52.2351" y2="32.37865" width="0.3048" layer="1"/>
-<wire x1="52.2351" y1="32.37865" x2="51.59375" y2="33.02" width="0.3048" layer="1"/>
-<wire x1="51.59375" y1="33.02" x2="51.59375" y2="35.21055" width="0.3048" layer="1"/>
-<wire x1="51.59375" y1="35.21055" x2="51.4858" y2="35.3185" width="0.3048" layer="1"/>
+<contactref element="U$1" pad="P$2"/>
+<wire x1="50.008" y1="26.935" x2="51.4858" y2="35.3185" width="0" layer="19" extent="1-1"/>
 </signal>
 <signal name="WS_CS">

Commit message: Finished rev 1.2.1
Parts:
- removed BNO180: BMP180, SparkFun-Sensors:BMP180
- added C1: 6.8nF, SparkFun-Passives:0805
- added C6, C9: .1uF, SparkFun-Passives:0805
- C2: value 10uF -> .1uF
- C5: value 4.7uF -> 120nF
- moved C3 23.4 mm to (37.8, 45.8), flipped to the top
- moved R7 21.2 mm to (57.2, 52.8), flipped to the bottom
- moved R8 20.0 mm to (59.1, 52.7), flipped to the bottom, turned to 90 degrees
- moved W25Q128FV 15.9 mm to (38.8, 39.8), flipped to the top, turned to 90 degrees
- moved C7 9.26 mm to (48.5, 39.4), flipped to the bottom, turned to 90 degrees
- moved U$1 8.66 mm to (48.8, 34.7), flipped to the bottom
- moved C5 7.88 mm to (46.1, 48.5), turned to 90 degrees
- moved C2 7.24 mm to (51.4, 56.1)
- moved BNO055 4.73 mm to (53.0, 52.6)
- moved C8 1.28 mm to (50.6, 39.4), turned to 90 degrees
- moved MCU 1.08 mm to (48.8, 39.3)
- moved C14 0.40 mm to (43.3, 56.8)
- moved D1 0.39 mm to (59.4, 48.6)
Connections:
- net N$6 renamed GPS-LED
- net GND: now also C1.1, C6.2, C9.1, U$1.P$4; no longer BNO180.7, U$1.P$3
- net ISP: now also U$1.P$6; no longer U$1.P$1
- net LPC_RX: now also U$1.P$1; no longer U$1.P$6
- net LPC_TX: now also U$1.P$2; no longer U$1.P$5
- net RESET: now also U$1.P$5; no longer U$1.P$2
- net SCL: now also R7.2; no longer BNO180.5, R8.2
- net SDA: now also R8.1; no longer BNO180.6, R7.2
- net VCC: now also C1.2, C6.1, C9.2, R8.2, U$1.P$3; no longer BNO180.2, BNO180.3, R8.1, U$1.P$4
Routing:
- net SCL: track 46.7 -> 21.1 mm, vias 4 -> 3
- net WS_CS: track 4.77 -> 23.6 mm, vias 1 -> 0
- net WS_DO: track 8.64 -> 22.4 mm, vias 1 -> 2
- net WS_DI: track 5.91 -> 14.2 mm, vias 1 -> 0
- net LPC_TX: track 21.9 -> 28.3 mm
- net LPC_RX: track 20.8 -> 25.8 mm
- net SDA: track 22.2 -> 17.4 mm, vias 3 -> 1
- net RESET: track 0.00 -> 4.61 mm, vias 0 -> 1
- net VCC: track 88.4 -> 84.5 mm
- net N$2: track 3.70 -> 1.84 mm
- net LPC_LED: track 7.84 -> 9.61 mm
- net GND: track 4.43 -> 5.57 mm, vias 0 -> 1
- net V_BATT: track 14.4 -> 13.9 mm
- net ISP: track 5.16 -> 4.62 mm, vias 0 -> 1
- net WS_SCK: track 11.9 -> 12.2 mm, vias 1 -> 0
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Other:
- board size 25.5 x 36.7 mm -> 25.4 x 36.7 mm

Commit message: Initial commit for QFN Package
Parts:
- removed MCU: LPC1112FD20/102, NXP_60_26022015:SOT163-1
- added U2: LPC1114FHI33/303, NXP_60_26022015:SOT617-3
- moved W25Q128FV 10.1 mm to (48.5, 43.0), turned to 180 degrees
Connections:
- new net VDD(IO): U2.6
- net GND: now also U2.33; no longer MCU.16
- net ISP: no longer MCU.18
- net LPC_LED: no longer MCU.3
- net LPC_RX: now also U2.13; no longer MCU.11
- net LPC_TX: now also U2.14; no longer MCU.12
- net RESET: now also U2.2; no longer MCU.17
- net SCL: now also U2.10; no longer MCU.20
- net SDA: now also U2.11; no longer MCU.5
- net VCC: now also U2.29; no longer MCU.15
- net WS_CS: no longer MCU.19
- net WS_DI: no longer MCU.2
- net WS_DO: no longer MCU.1
- net WS_SCK: now also U2.15; no longer MCU.6
Routing:
- net VCC: track 84.5 -> 28.7 mm, vias 3 -> 0
- net LPC_TX: track 28.3 -> 0.00 mm, vias 2 -> 0
- net LPC_RX: track 25.8 -> 0.00 mm, vias 2 -> 0
- net WS_CS: track 23.6 -> 0.00 mm
- net WS_DO: track 22.4 -> 0.00 mm, vias 2 -> 0
- net SCL: track 21.1 -> 1.84 mm, vias 3 -> 0
- net SDA: track 17.4 -> 0.00 mm, vias 1 -> 0
- net GPS-LED: track 16.9 -> 0.00 mm
- net WS_DI: track 14.2 -> 0.00 mm
- net N$10: track 12.4 -> 0.00 mm
- net WS_SCK: track 12.2 -> 0.00 mm
- net LPC_LED: track 9.61 -> 0.00 mm
- net N$4: track 6.35 -> 0.00 mm
- net ISP: track 4.62 -> 0.00 mm, vias 1 -> 0
- net RESET: track 4.61 -> 0.00 mm, vias 1 -> 0
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
Commit message: Fixup
Parts:
- removed U2: LPC1114FHI33/303, NXP_60_26022015:SOT617-3
- added MCU: LPC1114FHI33/302, NXP_60_26022015:SOT617-3
- moved C6 39.4 mm to (84.9, 67.7), turned to 0 degrees
- moved C2 38.2 mm to (88.5, 64.8), turned to 270 degrees
- moved C3 37.1 mm to (73.8, 37.0), turned to 270 degrees
- moved C4 36.2 mm to (73.2, 57.9), flipped to the bottom
- moved FB1 35.4 mm to (72.8, 60.6), flipped to the bottom, turned to 180 degrees
- moved U$1 35.1 mm to (79.6, 51.6), flipped to the top
- moved BNO055 33.7 mm to (85.0, 63.2), turned to 0 degrees
- moved MTK339 31.5 mm to (79.6, 62.9)
- moved BAT_CON 31.0 mm to (73.4, 70.5)
- moved R7 28.7 mm to (85.2, 59.0), turned to 0 degrees
- moved R8 26.4 mm to (85.2, 57.1), turned to 180 degrees
- moved W25Q128FV 21.0 mm to (68.7, 37.2)
- moved C5 12.6 mm to (58.7, 48.5)
- moved C7 10.6 mm to (57.5, 45.0), turned to 270 degrees
- moved C1 10.4 mm to (58.7, 51.8), turned to 270 degrees
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Connections:
- net GND: now also MCU.33; no longer U2.33
- net ISP: now also MCU.3
- net LPC_RX: now also MCU.31; no longer U2.13
- net LPC_TX: now also MCU.32; no longer U2.14
- net RESET: now also MCU.2; no longer U2.2
- net SCL: now also MCU.10; no longer U2.10
- net SDA: now also MCU.11; no longer U2.11
- net VCC: now also MCU.29; no longer U2.29
- net VDD(IO): now also MCU.6; no longer U2.6
- net WS_CS: now also MCU.8
- net WS_DI: now also MCU.18
- net WS_DO: now also MCU.17
- net WS_SCK: now also MCU.15; no longer U2.15
Routing:
- net VCC: track 28.7 -> 13.7 mm
- net V_BATT: track 13.9 -> 0.10 mm
- net N$3: track 3.11 -> 0.00 mm

Commit message: Initial Revision for QFN packages
Parts:
- removed BAT_CON: 53261-02, con-molex:53261-02
- removed C4, C9: .1uF, SparkFun-Passives:0805
- removed D2: GREEN, SparkFun-LED:LED-1206
- removed FB1: GetValue, microbuilder:0805
- removed JP2: (no value), microbuilder:JUMPER2
- removed MTK339: (no value), adafruit:FGPMMOPA6H
- removed U4: MIC2505 3.3, SparkFun-PowerIC:SOT23-5
- removed W25Q128FV: (no value), Matts-Parts:8-SOIC
- added FRAME1: FRAME-LEDGER, SparkFun-Aesthetics:CREATIVE_COMMONS
- added MIC5205: 3.3, SparkFun-PowerIC:SOT23-5
- added R2: 1M, SparkFun-Passives:0603-RES
- added R3: 330, SparkFun-Passives:0603-RES
- added S2: SWITCH-MOMENTARY-2SMD-3, SparkFun-Electromechanical:TACTILE_SWITCH_SMD-3
- added U$2: UBLOX_MAX, Ava:UBLOX_MAX
- added U$3: ANTENNA2SMD3, SparkFun-RF:ANTENNA-CHIP4
- added W25QWSON: (no value), Matts-Parts:WSON-8-PAD
- C1, C14, C2, C3, C5, C6, C7, C8: device SparkFun-Passives:0805 -> SparkFun-Passives:0603-CAP
- C15: value .1uF -> 2.2uF; device SparkFun-Passives:0805 -> SparkFun-Passives:0603-CAP
- D1: value PURPLE -> (none); device SparkFun-LED:LED-1206 -> SparkFun-LED:LED-0603
- R1, R4: value 330 -> 10K; device SparkFun-Passives:0805 -> SparkFun-Passives:0603-RES
- R7, R8: device SparkFun-Passives:0805 -> SparkFun-Passives:0603-RES
- moved MCU 78.2 mm to (11.4, 17.1), turned to 90 degrees
- moved U$1 77.7 mm to (13.7, 10.5)
- moved C6 77.5 mm to (14.9, 34.4)
- moved R7 77.0 mm to (15.9, 25.5)
- moved R8 76.9 mm to (15.8, 23.8)
- moved C2 76.8 mm to (19.1, 32.1)
- moved BNO055 76.7 mm to (15.7, 30.4)
- moved C3 69.9 mm to (6.80, 17.4), turned to 90 degrees
- moved R1 65.9 mm to (16.4, 10.9), flipped to the bottom, turned to 0 degrees
- moved C15 60.2 mm to (16.4, 9.22), turned to 180 degrees
- moved C14 59.7 mm to (11.5, 6.46), turned to 270 degrees
- moved R4 56.1 mm to (7.62, 30.1), flipped to the bottom, turned to 180 degrees
- moved D1 53.0 mm to (18.8, 22.4), turned to 0 degrees
- moved C5 51.0 mm to (10.6, 31.3)
- moved C1 50.6 mm to (12.4, 31.3), turned to 90 degrees
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Connections:
- removed net GPS-LED: D2.A, MTK339.P$5
- removed net LPC_LED: D1.A
- removed net N$10: JP2.2, MTK339.P$1
- removed net N$3: D1.C, R4.2
- removed net N$4: C4.1, FB1.1, JP2.1
- removed net N$9: D2.C, R1.1
- removed net VDD(IO): MCU.6
- removed net V_BATT: BAT_CON.2, C14.2, U4.1, U4.3
- new net BAT_MONITOR: MCU.24, R1.1, R2.2
- new net BTN: MCU.20, R4.1, S2.4
- new net LED: D1.A, MCU.25
- new net N$1: U$2.11_RF_IN, U$3.SIG
- new net N$5: D1.C, R3.2
- new net VIN: C14.2, MIC5205.1, MIC5205.3, R1.2, U$1.P$3
- net GND: now also MIC5205.2, R2.1, R3.1, S2.1, U$2.10_GND, U$2.12_GND, U$2.1_GND, W25QWSON.4; no longer BAT_CON.1, C4.2, C9.1, MTK339.P$12, MTK339.P$19, MTK339.P$3, MTK339.P$8, R1.2, R4.1, U4.2, W25Q128FV.4
- net LPC_RX: no longer MTK339.P$9
- net LPC_TX: no longer MTK339.P$10
- net SCL: now also U$2.17_SCL2
- net SDA: now also U$2.16_SDA2
- net VCC: now also MCU.6, MIC5205.5, R4.2, U$2.6_V_BCKP, U$2.7_VCC_IO, U$2.8_VCC, U$2.9_V_RESET, W25QWSON.3, W25QWSON.7, W25QWSON.8; no longer C9.2, FB1.2, U$1.P$3, U4.5, W25Q128FV.3, W25Q128FV.7, W25Q128FV.8
- net WS_CS: now also W25QWSON.1; no longer W25Q128FV.1
- net WS_DI: now also W25QWSON.5; no longer W25Q128FV.5
- net WS_DO: now also W25QWSON.2; no longer W25Q128FV.2
- net WS_SCK: now also W25QWSON.6; no longer W25Q128FV.6
Routing:
- net VCC: track 13.7 -> 84.4 mm, vias 0 -> 4
- net SDA: track 0.00 -> 24.2 mm, vias 0 -> 1
- net SCL: track 1.84 -> 22.7 mm, vias 0 -> 2
- net WS_DO: track 0.00 -> 16.8 mm, vias 0 -> 1
- net VIN: track 0.00 -> 16.0 mm, vias 0 -> 2
- net BTN: track 0.00 -> 14.1 mm, vias 0 -> 2
- net WS_CS: track 0.00 -> 10.8 mm, vias 0 -> 1
- net LPC_RX: track 0.00 -> 6.65 mm, vias 0 -> 1
- net LED: track 0.00 -> 6.23 mm, vias 0 -> 1
- net LPC_TX: track 0.00 -> 5.21 mm, vias 0 -> 1
- net ISP: track 0.00 -> 4.51 mm, vias 0 -> 1
- net RESET: track 0.00 -> 4.12 mm, vias 0 -> 1
- net WS_SCK: track 0.00 -> 3.63 mm, vias 0 -> 1
- net N$1: track 0.00 -> 3.58 mm
- net N$9: track 2.95 -> 0.00 mm
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Other:
- board size 25.4 x 36.7 mm -> 16.3 x 37.7 mm
- board text added: "ProSense Rev1.2"
- board text removed: "ProSense Rev1.1"
