File: ProSense.sch (EAGLE design)
At the start: 26 parts, among them U2 LPC1114FHI33/303, U4 MIC2505 3.3

Commit message: Fixup
Parts:
- removed U2: LPC1114FHI33/303, NXP_60_26022015:LPC1114FHI33/303
- added MCU: LPC1114FHI33/302, NXP_60_26022015:LPC1114FHI33/302
Connections:
- net GND: now also MCU.VSS; no longer U2.VSS
- net ISP: now also MCU.PIO0_1/CLKOUT/CT32B0_MAT2
- net LPC_RX: now also MCU.PIO1_6/RXD/CT32B0_MAT0; no longer U2.PIO3_4/CT16B0_CAP1/RXD
- net LPC_TX: now also MCU.PIO1_7/TXD/CT32B0_MAT1; no longer U2.PIO3_5/CT16B1_CAP1/TXD
- net RESET: now also MCU.!RESET!/PIO0_0; no longer U2.!RESET!/PIO0_0
- net SCL: now also MCU.PIO0_4/SCL; no longer U2.PIO0_4/SCL
- net SDA: now also MCU.PIO0_5/SDA; no longer U2.PIO0_5/SDA
- net VCC: now also MCU.VDD(3V3); no longer U2.VDD(3V3)
- net WS_CS: now also MCU.PIO0_2/SSEL0/CT16B0_CAP0
- net WS_DI: now also MCU.PIO0_9/MOSI0/CT16B0_MAT1
- net WS_DO: now also MCU.PIO0_8/MISO0/CT16B0_MAT0
- net WS_SCK: now also MCU.PIO0_6/SCK0; no longer U2.PIO0_6/SCK0
Other:
- moved on the sheet: C7, C8
Changed lines of the file:
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@@
 <part name="C9" library="SparkFun-Passives" deviceset="CAP" device="0805" value=".1uF"/>
 <part name="GND12" library="SparkFun-Aesthetics" deviceset="GND" device=""/>
-<part name="U2" library="NXP_60_26022015" deviceset="LPC1114FHI33/303" device=""/>
+<part name="MCU" library="NXP_60_26022015" deviceset="LPC1114FHI33/302" device=""/>
 </parts>
 <sheets>
@@
 <attribute name="VALUE" x="85.979" y="45.339" size="1.778" layer="96" rot="MR180"/>
 </instance>
-<instance part="C8" gate="G$1" x="-119.38" y="-7.62" smashed="yes" rot="MR0">
-<attribute name="NAME" x="-126.619" y="-7.366" size="1.778" layer="95" rot="MR90"/>
-<attribute name="VALUE" x="-124.079" y="-8.636" size="1.778" layer="96" rot="MR90"/>
-</instance>
-<instance part="GND28" gate="1" x="-119.38" y="-17.78" rot="MR0"/>
-<instance part="SUPPLY9" gate="G$1" x="-119.38" y="0" smashed="yes" rot="MR0">
-<attribute name="VALUE" x="-120.904" y="1.016" size="1.778" layer="96" rot="MR0"/>
+<instance part="C8" gate="G$1" x="-10.16" y="76.2" smashed="yes" rot="MR0">
+<attribute name="NAME" x="-17.399" y="76.454" size="1.778" layer="95" rot="MR90"/>
+<attribute name="VALUE" x="-14.859" y="75.184" size="1.778" layer="96" rot="MR90"/>
+</instance>
+<instance part="GND28" gate="1" x="-10.16" y="66.04" rot="MR0"/>
+<instance part="SUPPLY9" gate="G$1" x="-10.16" y="83.82" smashed="yes" rot="MR0">
+<attribute name="VALUE" x="-11.684" y="84.836" size="1.778" layer="96" rot="MR0"/>
 </instance>
 <instance part="SUPPLY11" gate="G$1" x="-81.28" y="121.92" rot="MR0"/>
@@
 </instance>
 <instance part="SUPPLY7" gate="G$1" x="43.18" y="48.006"/>
-<instance part="C7" gate="G$1" x="-132.08" y="-7.62" smashed="yes" rot="MR0">
-<attribute name="NAME" x="-139.319" y="-7.366" size="1.778" layer="95" rot="MR90"/>
-<attribute name="VALUE" x="-136.779" y="-8.636" size="1.778" layer="96" rot="MR90"/>
+<instance part="C7" gate="G$1" x="-22.86" y="76.2" smashed="yes" rot="MR0">
+<attribute name="NAME" x="-30.099" y="76.454" size="1.778" layer="95" rot="MR90"/>
+<attribute name="VALUE" x="-27.559" y="75.184" size="1.778" layer="96" rot="MR90"/>
 </instance>
 <instance part="C9" gate="G$1" x="-68.58" y="109.22" smashed="yes" rot="R180">
@@
 </instance>
 <instance part="GND12" gate="1" x="-68.58" y="96.52"/>
-<instance part="U2" gate="G$1" x="-60.96" y="17.78"/>
+<instance part="MCU" gate="G$1" x="45.72" y="99.06"/>
 </instances>
 <busses>
@@
 </segment>
 <segment>
-<wire x1="-106.68" y1="-2.54" x2="-119.38" y2="-2.54" width="0.1524" layer="91"/>
-<wire x1="-119.38" y1="-2.54" x2="-119.38" y2="0" width="0.1524" layer="91"/>
+<wire x1="0" y1="81.28" x2="-10.16" y2="81.28" width="0.1524" layer="91"/>
+<wire x1="-10.16" y1="81.28" x2="-10.16" y2="83.82" width="0.1524" layer="91"/>
 <pinref part="SUPPLY9" gate="G$1" pin="VCC"/>
 <pinref part="C8" gate="G$1" pin="1"/>
-<junction x="-119.38" y="-2.54"/>
+<junction x="-10.16" y="81.28"/>
 <pinref part="C7" gate="G$1" pin="1"/>
-<wire x1="-132.08" y1="-2.54" x2="-119.38" y2="-2.54" width="0.1524" layer="91"/>
-<pinref part="U2" gate="G$1" pin="VDD(3V3)"/>
+<wire x1="-22.86" y1="81.28" x2="-10.16" y2="81.28" width="0.1524" layer="91"/>
+<pinref part="MCU" gate="G$1" pin="VDD(3V3)"/>
 </segment>
 <segment>
@@
 </segment>
 <segment>
-<wire x1="-106.68" y1="-7.62" x2="-114.3" y2="-7.62" width="0.1524" layer="91"/>
-<wire x1="-114.3" y1="-7.62" x2="-114.3" y2="-10.16" width="0.1524" layer="91"/>
+<wire x1="0" y1="76.2" x2="-5.08" y2="76.2" width="0.1524" layer="91"/>
+<wire x1="-5.08" y1="76.2" x2="-5.08" y2="73.66" width="0.1524" layer="91"/>
 <pinref part="C8" gate="G$1" pin="2"/>
-<wire x1="-114.3" y1="-10.16" x2="-119.38" y2="-10.16" width="0.1524" layer="91"/>
+<wire x1="-5.08" y1="73.66" x2="-10.16" y2="73.66" width="0.1524" layer="91"/>
 <pinref part="GND28" gate="1" pin="GND"/>
-<wire x1="-119.38" y1="-10.16" x2="-119.38" y2="-15.24" width="0.1524" layer="91"/>
-<junction x="-119.38" y="-10.16"/>
+<wire x1="-10.16" y1="73.66" x2="-10.16" y2="68.58" width="0.1524" layer="91"/>
+<junction x="-10.16" y="73.66"/>
 <pinref part="C7" gate="G$1" pin="2"/>
-<wire x1="-132.08" y1="-10.16" x2="-119.38" y2="-10.16" width="0.1524" layer="91"/>
-<pinref part="U2" gate="G$1" pin="VSS"/>
+<wire x1="-22.86" y1="73.66" x2="-10.16" y2="73.66" width="0.1524" layer="91"/>
+<pinref part="MCU" gate="G$1" pin="VSS"/>
 </segment>
 <segment>
@@
 <net name="SDA" class="0">
 <segment>
-<wire x1="-106.68" y1="25.4" x2="-119.38" y2="25.4" width="0.1524" layer="91"/>
-<label x="-116.84" y="25.4" size="1.778" layer="95"/>
-<pinref part="U2" gate="G$1" pin="PIO0_5/SDA"/>
+<wire x1="0" y1="109.22" x2="-10.16" y2="109.22" width="0.1524" layer="91"/>
+<label x="-10.16" y="109.22" size="1.778" layer="95"/>
+<pinref part="MCU" gate="G$1" pin="PIO0_5/SDA"/>
 </segment>
 <segment>
@@
 <net name="SCL" class="0">
 <segment>
-<wire x1="-106.68" y1="27.94" x2="-119.38" y2="27.94" width="0.1524" layer="91"/>
-<label x="-116.84" y="27.94" size="1.778" layer="95"/>
-<pinref part="U2" gate="G$1" pin="PIO0_4/SCL"/>
+<wire x1="0" y1="111.76" x2="-10.16" y2="111.76" width="0.1524" layer="91"/>
+<label x="-10.16" y="111.76" size="1.778" layer="95"/>
+<pinref part="MCU" gate="G$1" pin="PIO0_4/SCL"/>
 </segment>
 <segment>
@@
 </segment>
 <segment>
-<wire x1="-15.24" y1="-2.54" x2="-2.54" y2="-2.54" width="0.1524" layer="91"/>
-<label x="-12.7" y="-2.54" size="1.778" layer="95"/>
-<pinref part="U2" gate="G$1" pin="PIO3_4/CT16B0_CAP1/RXD"/>
+<pinref part="MCU" gate="G$1" pin="PIO1_6/RXD/CT32B0_MAT0"/>
+<wire x1="91.44" y1="106.68" x2="104.14" y2="106.68" width="0.1524" layer="91"/>
+<label x="93.98" y="106.68" size="1.778" layer="95"/>
 </segment>
 </net>
@@
 </segment>
 <segment>
-<wire x1="-15.24" y1="-5.08" x2="-2.54" y2="-5.08" width="0.1524" layer="91"/>
-<label x="-12.7" y="-5.08" size="1.778" layer="95"/>
-<pinref part="U2" gate="G$1" pin="PIO3_5/CT16B1_CAP1/TXD"/>
+<pinref part="MCU" gate="G$1" pin="PIO1_7/TXD/CT32B0_MAT1"/>
+<wire x1="91.44" y1="104.14" x2="104.14" y2="104.14" width="0.1524" layer="91"/>
+<label x="93.98" y="104.14" size="1.778" layer="95"/>
 </segment>
 </net>
@@
 <net name="ISP" class="0">
 <segment>
-<wire x1="-25.4" y1="124.46" x2="-38.1" y2="124.46" width="0.1524" layer="91"/>
-<label x="-38.1" y="124.46" size="1.778" layer="95"/>
+<wire x1="0" y1="119.38" x2="-10.16" y2="119.38" width="0.1524" layer="91"/>
+<label x="-10.16" y="119.38" size="1.778" layer="95"/>
+<pinref part="MCU" gate="G$1" pin="PIO0_1/CLKOUT/CT32B0_MAT2"/>
 </segment>
 <segment>
@@
 <net name="RESET" class="0">
 <segment>
-<wire x1="-121.92" y1="38.1" x2="-106.68" y2="38.1" width="0.1524" layer="91"/>
-<label x="-119.38" y="38.1" size="1.778" layer="95"/>
-<pinref part="U2" gate="G$1" pin="!RESET!/PIO0_0"/>
+<wire x1="-10.16" y1="121.92" x2="0" y2="121.92" width="0.1524" layer="91"/>
+<label x="-10.16" y="121.92" size="1.778" layer="95"/>
+<pinref part="MCU" gate="G$1" pin="!RESET!/PIO0_0"/>
 </segment>
 <segment>
@@
 </segment>
 <segment>
-<wire x1="-25.4" y1="121.92" x2="-38.1" y2="121.92" width="0.1524" layer="91"/>
-<label x="-38.1" y="121.92" size="1.778" layer="95"/>
+<wire x1="0" y1="116.84" x2="-10.16" y2="116.84" width="0.1524" layer="91"/>
+<label x="-10.16" y="116.84" size="1.778" layer="95"/>
+<pinref part="MCU" gate="G$1" pin="PIO0_2/SSEL0/CT16B0_CAP0"/>
 </segment>
 </net>
@@
 </segment>
 <segment>
-<wire x1="-25.4" y1="109.22" x2="-38.1" y2="109.22" width="0.1524" layer="91"/>
-<label x="-38.1" y="109.22" size="1.778" layer="95"/>
+<wire x1="0" y1="101.6" x2="-10.16" y2="101.6" width="0.1524" layer="91"/>
+<label x="-10.16" y="101.6" size="1.778" layer="95"/>
+<pinref part="MCU" gate="G$1" pin="PIO0_8/MISO0/CT16B0_MAT0"/>
 </segment>
 </net>
@@
 </segment>
 <segment>
-<wire x1="-106.68" y1="22.86" x2="-119.38" y2="22.86" width="0.1524" layer="91"/>
-<label x="-116.84" y="22.86" size="1.778" layer="95"/>
-<pinref part="U2" gate="G$1" pin="PIO0_6/SCK0"/>
+<wire x1="0" y1="106.68" x2="-10.16" y2="106.68" width="0.1524" layer="91"/>
+<label x="-10.16" y="106.68" size="1.778" layer="95"/>
+<pinref part="MCU" gate="G$1" pin="PIO0_6/SCK0"/>
 </segment>
 </net>
@@
 </segment>
 <segment>
-<wire x1="-25.4" y1="106.68" x2="-38.1" y2="106.68" width="0.1524" layer="91"/>
-<label x="-38.1" y="106.68" size="1.778" layer="95"/>
+<wire x1="0" y1="99.06" x2="-10.16" y2="99.06" width="0.1524" layer="91"/>
+<label x="-10.16" y="99.06" size="1.778" layer="95"/>
+<pinref part="MCU" gate="G$1" pin="PIO0_9/MOSI0/CT16B0_MAT1"/>
 </segment>
 </net>
@@
 </segment>
 <segment>
-<wire x1="-114.3" y1="12.7" x2="-127" y2="12.7" width="0.1524" layer="91"/>
-<label x="-127" y="12.7" size="1.778" layer="95"/>
-</segment>
-</net>
+<wire x1="-5.08" y1="91.44" x2="-17.78" y2="91.44" width="0.1524" layer="91"/>
+<label x="-17.78" y="91.44" size="1.778" layer="95"/>
+</segment>
+</net>

Commit message: Initial Revision for QFN packages
Parts:
- removed BAT_CON: 53261-02, con-molex:53261-02
- removed C4, C9: .1uF, SparkFun-Passives:CAP0805
- removed D2: GREEN, SparkFun-LED:LED-GREENLARGE
- removed FB1: GetValue, microbuilder:FERRITE0805
- removed JP2: (no value), microbuilder:JUMPER2
- removed MTK339: (no value), adafruit:GPS_FGPMMOPA6H
- removed U4: MIC2505 3.3, SparkFun-PowerIC:MIC52053.3V
- removed W25Q128FV: (no value), Matts-Parts:W25Q128FV
- added FRAME1: FRAME-LEDGER, SparkFun-Aesthetics:FRAME-LEDGER
- added MIC5205: 3.3, SparkFun-PowerIC:MIC52053.3V
- added R2: 1M, SparkFun-Passives:RESISTOR0603-RES
- added R3: 330, SparkFun-Passives:RESISTOR0603-RES
- added S2: SWITCH-MOMENTARY-2SMD-3, SparkFun-Electromechanical:SWITCH-MOMENTARY-2SMD-3
- added U$2: UBLOX_MAX, Ava:UBLOX_MAX
- added U$3: ANTENNA2SMD3, SparkFun-RF:ANTENNA2SMD3
- added W25QWSON: (no value), Matts-Parts:W25Q128FVWSON
- C1, C14, C2, C3, C5, C6, C7, C8: device SparkFun-Passives:CAP0805 -> SparkFun-Passives:CAP0603-CAP
- C15: value .1uF -> 2.2uF; device SparkFun-Passives:CAP0805 -> SparkFun-Passives:CAP0603-CAP
- D1: value PURPLE -> (none); device SparkFun-LED:LED-PURPLE1206 -> SparkFun-LED:LED0603
- R1, R4: value 330 -> 10K; device SparkFun-Passives:RESISTOR0805-RES -> SparkFun-Passives:RESISTOR0603-RES
- R7, R8: device SparkFun-Passives:RESISTOR0805-RES -> SparkFun-Passives:RESISTOR0603-RES
Connections:
- removed net GPS-LED: D2.A, MTK339.3D-FIX
- removed net LPC_LED: D1.A
- removed net N$10: JP2.2, MTK339.VCC
- removed net N$3: D1.C, R4.2
- removed net N$4: C4.1, FB1.P$1, JP2.1
- removed net N$9: D2.C, R1.1
- removed net V_BATT: BAT_CON-2.S, C14.2, U4.EN, U4.IN
- new net BAT_MONITOR: MCU.R/PIO1_2/AD3/CT32B1_MAT1, R1.1, R2.2
- new net BTN: MCU.PIO1_10/AD6/CT16B1_MAT1, R4.1, S2.2
- new net LED: D1.A, MCU.SWDIO/PIO1_3/AD4/CT32B1_MAT2
- new net N$1: U$2.11_RF_IN, U$3.SIGNAL
- new net N$5: D1.C, R3.2
- new net VIN: C14.2, MIC5205.EN, MIC5205.IN, R1.2, U$1.3
- net GND: now also MIC5205.GND, R2.1, R3.1, S2.1, U$2.10_GND, U$2.12_GND, U$2.1_GND, W25QWSON.GND; no longer BAT_CON-1.S, C4.2, C9.1, MTK339.GND@1, MTK339.GND@2, MTK339.GND@3, MTK339.GND@4, R1.2, R4.1, U4.GND, W25Q128FV.GND
- net LPC_RX: no longer MTK339.TX
- net LPC_TX: no longer MTK339.RX
- net SCL: now also U$2.17_SCL2
- net SDA: now also U$2.16_SDA2
- net VCC: now also MCU.VDD(IO), MIC5205.OUT, R4.2, U$2.6_V_BCKP, U$2.7_VCC_IO, U$2.8_VCC, U$2.9_V_RESET, W25QWSON.RESET, W25QWSON.VCC, W25QWSON.WP; no longer C9.2, FB1.P$2, U$1.3, U4.OUT, W25Q128FV.RESET, W25Q128FV.VCC, W25Q128FV.WP
- net WS_CS: now also W25QWSON.CS; no longer W25Q128FV.CS
- net WS_DI: now also W25QWSON.DI; no longer W25Q128FV.DI
- net WS_DO: now also W25QWSON.DO; no longer W25Q128FV.DO
- net WS_SCK: now also W25QWSON.CLK; no longer W25Q128FV.CLK
Other:
- moved on the sheet: BNO055, C1, C14, C15, C2, C3, C5, C6, C7, C8, D1, MCU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

Commit message: Fixed up a few things. Need to fix ground pads and holes for qfn
Parts:
- removed FRAME1: FRAME-LEDGER, SparkFun-Aesthetics:FRAME-LEDGER
Connections:
- net BAT_MONITOR: now also MCU.PIO1_11/AD7; no longer MCU.R/PIO1_2/AD3/CT32B1_MAT1
Changed lines of the file:
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@@
 <setting verticaltext="up"/>
 </settings>
-<grid distance="0.005" unitdist="inch" unit="inch" style="lines" multiple="1" display="no" altdistance="0.01" altunitdist="inch" altunit="inch"/>
+<grid distance="0.1" unitdist="inch" unit="inch" style="lines" multiple="1" display="no" altdistance="0.01" altunitdist="inch" altunit="inch"/>
 <layers>
 <layer number="1" name="Top" color="4" fill="1" visible="no" active="no"/>
@@
 <part name="SUPPLY3" library="SparkFun-Aesthetics" deviceset="VIN" device=""/>
 <part name="SUPPLY13" library="SparkFun-Aesthetics" deviceset="VIN" device=""/>
-<part name="FRAME1" library="SparkFun-Aesthetics" deviceset="FRAME-LEDGER" device=""/>
 <part name="S2" library="SparkFun-Electromechanical" deviceset="SWITCH-MOMENTARY-2" device="SMD-3"/>
 <part name="D1" library="SparkFun-LED" deviceset="LED" device="0603"/>
@@
 <instance part="SUPPLY3" gate="G$1" x="113.03" y="74.041"/>
 <instance part="SUPPLY13" gate="G$1" x="-116.332" y="7.366"/>
-<instance part="FRAME1" gate="G$1" x="-196.85" y="-104.648"/>
-<instance part="FRAME1" gate="G$2" x="133.35" y="-104.648"/>
 <instance part="S2" gate="G$1" x="-65.024" y="-54.102"/>
 <instance part="D1" gate="G$1" x="-95.377" y="-66.04" rot="R270"/>
@@
 </segment>
 <segment>
-<pinref part="MCU" gate="G$1" pin="R/PIO1_2/AD3/CT32B1_MAT1"/>
-<wire x1="76.835" y1="69.596" x2="84.455" y2="69.596" width="0.1524" layer="91"/>
-<wire x1="84.455" y1="69.596" x2="84.455" y2="69.977" width="0.1524" layer="91"/>
-</segment>
-</net>
+<wire x1="76.835" y1="46.736" x2="90.805" y2="46.736" width="0.1524" layer="91"/>
+<label x="77.978" y="44.45" size="1.778" layer="95"/>
+<pinref part="MCU" gate="G$1" pin="PIO1_11/AD7"/>
+</segment>
+</net>

Commit message: MTK3339 readded
Parts:
- removed U$2: UBLOX_MAX, Ava:UBLOX_MAX
- removed U$3: ANTENNA2SMD3, SparkFun-RF:ANTENNA2SMD3
- added 330: (no value), SparkFun-Passives:RESISTOR0603-RES
- added C4: 10uF, SparkFun-Passives:CAP0603-CAP
- added D2: (no value), SparkFun-LED:LED0603
- added FB1: (no value), microbuilder:FERRITE_0603MP
- added S1: (no value), SparkFun-Electromechanical:SWITCH-SPDTSMD2
- added U1: (no value), adafruit:GPS_FGPMMOPA6H
Connections:
- new net N$3: C4.1, S1.O
- new net N$4: D2.A, U1.3D-FIX
- new net N$6: C4.2, U1.VCC
- new net N$7: FB1.P$1, S1.P
- net GND: now also 330.1, U1.GND@1, U1.GND@2, U1.GND@3, U1.GND@4; no longer U$2.10_GND, U$2.12_GND, U$2.1_GND
- net LPC_RX: now also U1.TX
- net LPC_TX: now also U1.RX
- net N$1: now also 330.2, D2.C; no longer U$2.11_RF_IN, U$3.SIGNAL
- net SCL: no longer U$2.17_SCL2
- net SDA: no longer U$2.16_SDA2
- net VCC: now also FB1.P$2; no longer U$2.6_V_BCKP, U$2.7_VCC_IO, U$2.8_VCC, U$2.9_V_RESET
