File: ProSense.sch (EAGLE design)
At the start: 24 parts

Commit message: Squash
Parts:
- added C4: .1uF, SparkFun-Passives:CAP0603-CAP
- added U$4: CON, Matts-Parts:CON
- renumbered D1 to LPCLED, U$3 to ANT
Connections:
- new net SIG: MCU.PIO2_0/!DTR!, U$4.SIG
- net GND: now also C4.1, U$4.GND
- net VCC: now also C4.2
- net VIN: now also U$4.VLED
Changed lines of the file:
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@@
 <setting verticaltext="up"/>
 </settings>
-<grid distance="0.1" unitdist="inch" unit="inch" style="lines" multiple="1" display="no" altdistance="0.01" altunitdist="inch" altunit="inch"/>
+<grid distance="0.005" unitdist="inch" unit="inch" style="lines" multiple="1" display="no" altdistance="0.01" altunitdist="inch" altunit="inch"/>
 <layers>
 <layer number="1" name="Top" color="4" fill="1" visible="no" active="no"/>
@@
 <part name="W25QWSON" library="Matts-Parts" deviceset="W25Q128FV" device="WSON"/>
 <part name="U$2" library="Ava" deviceset="UBLOX_MAX" device=""/>
-<part name="U$3" library="SparkFun-RF" deviceset="ANTENNA2" device="SMD3"/>
+<part name="ANT" library="SparkFun-RF" deviceset="ANTENNA2" device="SMD3"/>
 <part name="GND15" library="SparkFun-Aesthetics" deviceset="GND" device=""/>
 <part name="GND17" library="SparkFun-Aesthetics" deviceset="GND" device=""/>
@@
 <part name="SUPPLY13" library="SparkFun-Aesthetics" deviceset="VIN" device=""/>
 <part name="S2" library="SparkFun-Electromechanical" deviceset="SWITCH-MOMENTARY-2" device="SMD-3"/>
-<part name="D1" library="SparkFun-LED" deviceset="LED" device="0603"/>
+<part name="LPCLED" library="SparkFun-LED" deviceset="LED" device="0603"/>
 <part name="R3" library="SparkFun-Passives" deviceset="RESISTOR" device="0603-RES" value="330"/>
 <part name="GND1" library="SparkFun-Aesthetics" deviceset="GND" device=""/>
@@
 <part name="GND20" library="SparkFun-Aesthetics" deviceset="GND" device=""/>
 <part name="R4" library="SparkFun-Passives" deviceset="RESISTOR" device="0603-RES" value="10K"/>
+<part name="C4" library="SparkFun-Passives" deviceset="CAP" device="0603-CAP" value=".1uF"/>
+<part name="GND12" library="SparkFun-Aesthetics" deviceset="GND" device=""/>
+<part name="U$4" library="Matts-Parts" deviceset="CON" device=""/>
+<part name="GND22" library="SparkFun-Aesthetics" deviceset="GND" device=""/>
+<part name="SUPPLY14" library="SparkFun-Aesthetics" deviceset="VIN" device=""/>
 </parts>
 <sheets>
@@
 <instance part="W25QWSON" gate="G$1" x="-125.73" y="51.816"/>
 <instance part="U$2" gate="G$1" x="55.118" y="120.142"/>
-<instance part="U$3" gate="G$1" x="13.462" y="130.302" smashed="yes" rot="R90">
+<instance part="ANT" gate="G$1" x="13.462" y="130.302" smashed="yes" rot="R90">
 <attribute name="NAME" x="3.302" y="126.492" size="1.778" layer="95" rot="R90"/>
 <attribute name="VALUE" x="5.842" y="121.412" size="1.778" layer="96" rot="R90"/>
@@
 <instance part="GND17" gate="1" x="15.748" y="135.382" rot="R270"/>
 <instance part="GND19" gate="1" x="93.218" y="94.742" rot="R90"/>
-<instance part="SUPPLY5" gate="G$1" x="98.298" y="127.762" rot="R270"/>
+<instance part="SUPPLY5" gate="G$1" x="98.298" y="131.318"/>
 <instance part="R1" gate="G$1" x="-116.332" y="-0.762" rot="R90"/>
 <instance part="R2" gate="G$1" x="-116.332" y="-20.828" rot="R90"/>
@@
 <instance part="SUPPLY3" gate="G$1" x="113.03" y="74.041"/>
 <instance part="SUPPLY13" gate="G$1" x="-116.332" y="7.366"/>
-<instance part="S2" gate="G$1" x="-65.024" y="-54.102"/>
-<instance part="D1" gate="G$1" x="-95.377" y="-66.04" rot="R270"/>
+<instance part="S2" gate="G$1" x="-65.024" y="-54.102" smashed="yes">
+<attribute name="NAME" x="-67.564" y="-51.562" size="1.778" layer="95"/>
+<attribute name="VALUE" x="-98.044" y="-49.022" size="1.778" layer="96"/>
+</instance>
+<instance part="LPCLED" gate="G$1" x="-95.377" y="-66.04" rot="R270"/>
 <instance part="R3" gate="G$1" x="-108.458" y="-71.12" rot="R90"/>
 <instance part="GND1" gate="1" x="-108.458" y="-84.836"/>
@@
 </instance>
 <instance part="R4" gate="G$1" x="-51.054" y="-47.498" rot="R90"/>
+<instance part="C4" gate="G$1" x="98.298" y="121.158" rot="R180"/>
+<instance part="GND12" gate="1" x="98.298" y="106.68"/>
+<instance part="U$4" gate="G$1" x="-86.36" y="119.38" rot="R90"/>
+<instance part="GND22" gate="1" x="-83.82" y="114.3"/>
+<instance part="SUPPLY14" gate="G$1" x="-76.2" y="127" rot="R270"/>
 </instances>
 <busses>
@@
 </segment>
 <segment>
-<pinref part="U$2" gate="G$1" pin="9_V_RESET"/>
-<wire x1="77.978" y1="135.382" x2="88.138" y2="135.382" width="0.1524" layer="91"/>
-<wire x1="88.138" y1="135.382" x2="88.138" y2="130.302" width="0.1524" layer="91"/>
-<pinref part="U$2" gate="G$1" pin="6_V_BCKP"/>
-<wire x1="88.138" y1="130.302" x2="88.138" y2="127.762" width="0.1524" layer="91"/>
-<wire x1="88.138" y1="127.762" x2="88.138" y2="125.222" width="0.1524" layer="91"/>
-<wire x1="88.138" y1="125.222" x2="88.138" y2="120.142" width="0.1524" layer="91"/>
-<wire x1="88.138" y1="120.142" x2="77.978" y2="120.142" width="0.1524" layer="91"/>
-<pinref part="U$2" gate="G$1" pin="7_VCC_IO"/>
-<wire x1="77.978" y1="125.222" x2="88.138" y2="125.222" width="0.1524" layer="91"/>
-<junction x="88.138" y="125.222"/>
-<pinref part="U$2" gate="G$1" pin="8_VCC"/>
-<wire x1="77.978" y1="130.302" x2="88.138" y2="130.302" width="0.1524" layer="91"/>
-<junction x="88.138" y="130.302"/>
-<wire x1="88.138" y1="127.762" x2="98.298" y2="127.762" width="0.1524" layer="91"/>
-<junction x="88.138" y="127.762"/>
-<pinref part="SUPPLY5" gate="G$1" pin="VCC"/>
-</segment>
-<segment>
 <pinref part="R4" gate="G$1" pin="2"/>
 <pinref part="SUPPLY10" gate="G$1" pin="VCC"/>
 <wire x1="-51.054" y1="-42.418" x2="-51.054" y2="-35.814" width="0.1524" layer="91"/>
+</segment>
+<segment>
+<pinref part="SUPPLY5" gate="G$1" pin="VCC"/>
+<pinref part="C4" gate="G$1" pin="2"/>
+<wire x1="98.298" y1="131.318" x2="98.298" y2="127.889" width="0.1524" layer="91"/>
+<pinref part="U$2" gate="G$1" pin="9_V_RESET"/>
+<pinref part="U$2" gate="G$1" pin="8_VCC"/>
+<wire x1="98.298" y1="127.889" x2="98.298" y2="123.698" width="0.1524" layer="91"/>
+<wire x1="77.978" y1="135.382" x2="77.978" y2="130.302" width="0.1524" layer="91"/>
+<pinref part="U$2" gate="G$1" pin="7_VCC_IO"/>
+<wire x1="77.978" y1="130.302" x2="77.978" y2="127.889" width="0.1524" layer="91"/>
+<junction x="77.978" y="130.302"/>
+<pinref part="U$2" gate="G$1" pin="6_V_BCKP"/>
+<wire x1="77.978" y1="127.889" x2="77.978" y2="125.222" width="0.1524" layer="91"/>
+<wire x1="77.978" y1="125.222" x2="77.978" y2="120.142" width="0.1524" layer="91"/>
+<junction x="77.978" y="125.222"/>
+<wire x1="77.978" y1="127.889" x2="98.298" y2="127.889" width="0.1524" layer="91"/>
+<junction x="77.978" y="127.889"/>
+<junction x="98.298" y="127.889"/>
 </segment>
 </net>
@@
 <pinref part="GND20" gate="1" pin="GND"/>
 </segment>
+<segment>
+<pinref part="C4" gate="G$1" pin="1"/>
+<pinref part="GND12" gate="1" pin="GND"/>
+<wire x1="98.298" y1="116.078" x2="98.298" y2="109.22" width="0.1524" layer="91"/>
+</segment>
+<segment>
+<pinref part="U$4" gate="G$1" pin="GND"/>
+<wire x1="-88.9" y1="119.38" x2="-83.82" y2="119.38" width="0.1524" layer="91"/>
+<wire x1="-83.82" y1="119.38" x2="-83.82" y2="116.84" width="0.1524" layer="91"/>
+<pinref part="GND22" gate="1" pin="GND"/>
+</segment>
 </net>
 <net name="N$2" class="0">
@@
 <segment>
 <pinref part="U$2" gate="G$1" pin="11_RF_IN"/>
-<pinref part="U$3" gate="G$1" pin="SIGNAL"/>
+<pinref part="ANT" gate="G$1" pin="SIGNAL"/>
 <wire x1="18.542" y1="130.302" x2="32.258" y2="130.302" width="0.1524" layer="91"/>
 </segment>
@@
 <pinref part="SUPPLY13" gate="G$1" pin="VIN"/>
 </segment>
+<segment>
+<pinref part="U$4" gate="G$1" pin="VLED"/>
+<wire x1="-88.9" y1="127" x2="-76.2" y2="127" width="0.1524" layer="91"/>
+<pinref part="SUPPLY14" gate="G$1" pin="VIN"/>
+</segment>
 </net>
 <net name="LED" class="0">
 <segment>
-<pinref part="D1" gate="G$1" pin="A"/>
+<pinref part="LPCLED" gate="G$1" pin="A"/>
 <wire x1="-92.837" y1="-66.04" x2="-84.074" y2="-66.04" width="0.1524" layer="91"/>
 <label x="-88.646" y="-65.659" size="1.778" layer="95"/>
@@
 <net name="N$5" class="0">
 <segment>
-<pinref part="D1" gate="G$1" pin="C"/>
+<pinref part="LPCLED" gate="G$1" pin="C"/>
 <wire x1="-100.457" y1="-66.04" x2="-108.458" y2="-66.04" width="0.1524" layer="91"/>
 <pinref part="R3" gate="G$1" pin="2"/>
@@
 <pinref part="R4" gate="G$1" pin="1"/>
 <wire x1="-51.054" y1="-54.102" x2="-51.054" y2="-52.578" width="0.1524" layer="91"/>
+<label x="-58.42" y="-53.34" size="1.778" layer="95"/>
 </segment>
 <segment>
@@
 </segment>
 </net>
+<net name="SIG" class="0">
+<segment>
+<pinref part="MCU" gate="G$1" pin="PIO2_0/!DTR!"/>
+<wire x1="76.835" y1="41.656" x2="87.884" y2="41.656" width="0.1524" layer="91"/>
+<wire x1="87.884" y1="41.656" x2="87.884" y2="41.783" width="0.1524" layer="91"/>
+<label x="80.899" y="41.656" size="1.778" layer="95"/>
+</segment>
+<segment>
+<pinref part="U$4" gate="G$1" pin="SIG"/>
+<wire x1="-88.9" y1="134.62" x2="-76.2" y2="134.62" width="0.1524" layer="91"/>
+<label x="-81.026" y="134.747" size="1.778" layer="95"/>
+</segment>
+</net>
